File: V2164tests.kicad_pcb (KiCad board)
At the start: 2 copper layers, 33 x 80 mm, 54 parts, among them J1 Conn_01x08, J2 Conn_01x08, J3 Conn_01x07, J4 Conn_01x07, U1 SSI2164, U2 TL074

Commit message: fixes v0.2
Parts:
- moved R1 6.00 mm to (104.5, 142.0)
- moved R15 4.59 mm to (85.5, 142.0)
- moved R14 4.22 mm to (90.0, 142.0)
- moved R4 3.37 mm to (99.6, 142.0)
Connections:
- RV1 pad 1: Net-(R4-Pad2) -> Net-(R1-Pad1)
- RV1 pad 3: Net-(R1-Pad1) -> Net-(R4-Pad2)
- RV2 pad 1: Net-(R15-Pad2) -> Net-(R14-Pad1)
- RV2 pad 3: Net-(R14-Pad1) -> Net-(R15-Pad2)
Routing:
- net +12V: track 106.7 -> 118.8 mm, vias 3 -> 4
- net -12V: track 114.3 -> 116.7 mm
- net Net-(R14-Pad1): track 5.35 -> 3.41 mm
- net Net-(R4-Pad2): track 5.25 -> 3.76 mm
- net Net-(R15-Pad2): track 4.32 -> 3.20 mm
- net Net-(R1-Pad1): track 4.27 -> 3.27 mm
- net /U10: track 36.5 -> 35.6 mm
Other:
- board text added: "CV 3+4"
- board text added: "v0.2"
- board text removed: "CV 2+4"
