File: V2164tests.kicad_sch (KiCad schematic)
At the start: 54 parts, among them J1 Conn_01x08, J2 Conn_01x08, J3 Conn_01x07, J4 Conn_01x07, U1 SSI2164, U2 TL074

Commit message: fixes v0.2
Connections:
- net at R4.2: now also RV1.3; no longer RV1.1
- net at R1.1: now also RV1.1; no longer RV1.3
- net at R14.1: now also RV2.1; no longer RV2.3
- net at R15.2: now also RV2.3; no longer RV2.1
Changed lines of the file:
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@@
+	)
+	(junction
+		(at 39.37 156.21)
+		(diameter 0)
+		(color 0 0 0 0)
 	)
 	(junction
@@
 	)
 	(junction
+		(at 81.28 163.83)
+		(diameter 0)
+		(color 0 0 0 0)
+	)
+	(junction
 		(at 62.23 88.9)
 		(diameter 0)
@@
 		(color 0 0 0 0)
 	)
+	(junction
+		(at 81.28 173.99)
+		(diameter 0)
+		(color 0 0 0 0)
+	)
 	(wire
 		(pts
@@
 	(wire
 		(pts
-			(xy 39.37 153.67) (xy 33.02 153.67)
-		)
-		(stroke
-			(width 0)
-			(type default)
-		)
-	)
-	(wire
-		(pts
 			(xy 48.26 160.02) (xy 44.45 160.02)
 		)
@@
 	(wire
 		(pts
+			(xy 81.28 163.83) (xy 81.28 166.37)
+		)
+		(stroke
+			(width 0)
+			(type default)
+		)
+	)
+	(wire
+		(pts
 			(xy 116.84 44.45) (xy 114.3 46.99)
 		)
@@
 	(wire
 		(pts
-			(xy 33.02 163.83) (xy 39.37 163.83)
-		)
-		(stroke
-			(width 0)
-			(type default)
-		)
-	)
-	(wire
-		(pts
 			(xy 91.44 93.98) (xy 91.44 88.9)
 		)
@@
 	(wire
 		(pts
+			(xy 36.83 156.21) (xy 39.37 156.21)
+		)
+		(stroke
+			(width 0)
+			(type default)
+		)
+	)
+	(wire
+		(pts
+			(xy 81.28 173.99) (xy 81.28 176.53)
+		)
+		(stroke
+			(width 0)
+			(type default)
+		)
+	)
+	(wire
+		(pts
 			(xy 100.33 46.99) (xy 100.33 40.64)
 		)
@@
 	(wire
 		(pts
-			(xy 33.02 153.67) (xy 33.02 163.83)
-		)
-		(stroke
-			(width 0)
-			(type default)
-		)
-	)
-	(wire
-		(pts
-			(xy 74.93 176.53) (xy 81.28 176.53)
-		)
-		(stroke
-			(width 0)
-			(type default)
-		)
-	)
-	(wire
-		(pts
 			(xy 172.72 44.45) (xy 161.29 44.45)
 		)
@@
 	(wire
 		(pts
-			(xy 39.37 166.37) (xy 36.83 166.37)
-		)
-		(stroke
-			(width 0)
-			(type default)
-		)
-	)
-	(wire
-		(pts
 			(xy 62.23 121.92) (xy 66.04 121.92)
 		)
@@
 	(wire
 		(pts
-			(xy 36.83 166.37) (xy 36.83 156.21)
-		)
-		(stroke
-			(width 0)
-			(type default)
-		)
-	)
-	(wire
-		(pts
 			(xy 95.25 135.89) (xy 63.5 135.89)
 		)
@@
 	(wire
 		(pts
-			(xy 78.74 173.99) (xy 78.74 163.83)
-		)
-		(stroke
-			(width 0)
-			(type default)
-		)
-	)
-	(wire
-		(pts
 			(xy 172.72 30.48) (xy 172.72 36.83)
 		)
@@
 	(wire
 		(pts
-			(xy 36.83 156.21) (xy 39.37 156.21)
-		)
-		(stroke
-			(width 0)
-			(type default)
-		)
-	)
-	(wire
-		(pts
 			(xy 120.65 140.97) (xy 120.65 129.54)
 		)
@@
 	(wire
 		(pts
-			(xy 81.28 166.37) (xy 74.93 166.37)
-		)
-		(stroke
-			(width 0)
-			(type default)
-		)
-	)
-	(wire
-		(pts
 			(xy 166.37 116.84) (xy 168.91 116.84)
 		)
@@
 	(wire
 		(pts
+			(xy 39.37 163.83) (xy 39.37 166.37)
+		)
+		(stroke
+			(width 0)
+			(type default)
+		)
+	)
+	(wire
+		(pts
 			(xy 154.94 87.63) (xy 152.4 87.63)
 		)
@@
 	(wire
 		(pts
-			(xy 74.93 166.37) (xy 74.93 176.53)
-		)
-		(stroke
+			(xy 39.37 153.67) (xy 39.37 156.21)
+		)
+		(stroke
